File: raspi_motherboard/untitled.kicad_sch (KiCad schematic)
At the start: 8 parts, among them U1 MCP2515-xST, U2 SN65HVD230, Y1 AMB8-12Mhz

Commit message: Commit missed element
Parts:
- renumbered C2 to C1, C1 to C2
