File: raspi_motherboard/untitled.kicad_sch (KiCad schematic)
At the start: 8 parts, among them U1 MCP2515-xST, U2 SN65HVD230, Y1 AMB8-12Mhz

Commit message: fix ERC/DRC (including short-circuits) + add flood fills
Parts:
- renumbered C2 to C1, C1 to C2
Connections:
- no-connect marks 0 -> 7

Commit message: [WiP] start putting refs in silkscreen
Parts:
- renumbered R_RESET2 to R1, R_CAN1 to R2, R_RESET1 to R3
Other:
- moved on the sheet: C1
Changed lines of the file:
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@@
-	)
-	(junction
-		(at 39.37 63.5)
-		(diameter 0)
-		(color 0 0 0 0)
 	)
 	(junction
@@
 	)
 	(junction
+		(at 34.29 55.88)
+		(diameter 0)
+		(color 0 0 0 0)
+	)
+	(junction
 		(at 71.12 72.39)
+		(diameter 0)
+		(color 0 0 0 0)
+	)
+	(junction
+		(at 44.45 72.39)
 		(diameter 0)
 		(color 0 0 0 0)
@@
 		(color 0 0 0 0)
 	)
-	(junction
-		(at 36.83 55.88)
-		(diameter 0)
-		(color 0 0 0 0)
-	)
 	(no_connect
 		(at 86.36 59.69)
@@
 	(wire
 		(pts
-			(xy 30.48 55.88) (xy 36.83 55.88)
+			(xy 44.45 72.39) (xy 71.12 72.39)
+		)
+		(stroke
+			(width 0)
+			(type default)
+		)
+	)
+	(wire
+		(pts
+			(xy 30.48 55.88) (xy 34.29 55.88)
 		)
 		(stroke
@@
 	(wire
 		(pts
+			(xy 46.99 55.88) (xy 46.99 57.15)
+		)
+		(stroke
+			(width 0)
+			(type default)
+		)
+	)
+	(wire
+		(pts
 			(xy 121.92 25.4) (xy 118.11 25.4)
 		)
@@
 	(wire
 		(pts
-			(xy 33.02 60.96) (xy 44.45 60.96)
-		)
-		(stroke
-			(width 0)
-			(type default)
-		)
-	)
-	(wire
-		(pts
-			(xy 39.37 63.5) (xy 39.37 59.69)
-		)
-		(stroke
-			(width 0)
-			(type default)
-		)
-	)
-	(wire
-		(pts
 			(xy 44.45 59.69) (xy 41.91 59.69)
 		)
@@
 	(wire
 		(pts
-			(xy 39.37 72.39) (xy 71.12 72.39)
-		)
-		(stroke
-			(width 0)
-			(type default)
-		)
-	)
-	(wire
-		(pts
-			(xy 36.83 55.88) (xy 36.83 59.69)
-		)
-		(stroke
-			(width 0)
-			(type default)
-		)
-	)
-	(wire
-		(pts
-			(xy 39.37 63.5) (xy 46.99 63.5)
-		)
-		(stroke
-			(width 0)
-			(type default)
-		)
-	)
-	(wire
-		(pts
 			(xy 121.92 48.26) (xy 121.92 50.8)
 		)
@@
 	(wire
 		(pts
-			(xy 44.45 59.69) (xy 44.45 60.96)
+			(xy 44.45 59.69) (xy 44.45 62.23)
 		)
 		(stroke
@@
 	(wire
 		(pts
-			(xy 39.37 72.39) (xy 39.37 63.5)
-		)
-		(stroke
-			(width 0)
-			(type default)
-		)
-	)
-	(wire
-		(pts
 			(xy 135.89 52.07) (xy 133.35 52.07)
 		)
@@
 	(wire
 		(pts
-			(xy 39.37 59.69) (xy 36.83 59.69)
-		)
-		(stroke
-			(width 0)
-			(type default)
-		)
-	)
-	(wire
-		(pts
 			(xy 30.48 48.26) (xy 30.48 49.53)
 		)
@@
 	(wire
 		(pts
+			(xy 46.99 57.15) (xy 34.29 57.15)
+		)
+		(stroke
+			(width 0)
+			(type default)
+		)
+	)
+	(wire
+		(pts
 			(xy 49.53 41.91) (xy 55.88 41.91)
 		)
@@
 	(wire
 		(pts
+			(xy 25.4 72.39) (xy 44.45 72.39)
+		)
+		(stroke
+			(width 0)
+			(type default)
+		)
+	)
+	(wire
+		(pts
 			(xy 71.12 26.67) (xy 71.12 29.21)
 		)
@@
 	(wire
 		(pts
+			(xy 34.29 55.88) (xy 34.29 57.15)
+		)
+		(stroke
+			(width 0)
+			(type default)
+		)
+	)
+	(wire
+		(pts
 			(xy 132.08 36.83) (xy 135.89 36.83)
 		)
@@
 	(wire
 		(pts
-			(xy 46.99 55.88) (xy 46.99 63.5)
-		)
-		(stroke
-			(width 0)
-			(type default)
-		)
-	)
-	(wire
-		(pts
 			(xy 71.12 72.39) (xy 71.12 69.85)
 		)
@@
 	(wire
 		(pts
+			(xy 34.29 55.88) (xy 36.83 55.88)
+		)
+		(stroke
+			(width 0)
+			(type default)
+		)
+	)
+	(wire
+		(pts
 			(xy 133.35 40.64) (xy 133.35 52.07)
 		)
@@
 	(wire
 		(pts
-			(xy 25.4 60.96) (xy 25.4 49.53)
+			(xy 25.4 49.53) (xy 25.4 72.39)
+		)
+		(stroke
+			(width 0)
+			(type default)
+		)
+	)
+	(wire
+		(pts
+			(xy 44.45 69.85) (xy 44.45 72.39)
 		)
 		(stroke
@@
 		(on_board yes)
 		(dnp no)
-		(fields_autoplaced yes)
-		(property "Reference" "R_RESET2"
+		(property "Reference" "R1"
 			(at 109.22 48.26 0)
 			(effects
@@
 			)
 		)
-		(property "Description" ""
-			(at 106.68 49.53 0)
-			(effects
-				(font
-					(size 1.27 1.27)
-				)
-				(hide yes)
+		(property "Description" "R_RESET2"
+			(at 104.648 49.53 90)
+			(effects
+				(font
+					(size 1.27 1.27)
+				)
 			)
 		)
@@
 			(project "power_motherboard"
 				(path "/e63e39d7-6ac0-4ffd-8aa3-1841a4541b55/fdc48edb-4989-401e-a47f-b3b658706075"
-					(reference "R_RESET2")
+					(reference "R1")
 					(unit 1)
 				)
@@
 		(on_board yes)
 		(dnp no)
-		(fields_autoplaced yes)
-		(property "Reference" "R_RESET1"
+		(property "Reference" "R3"
 			(at 92.71 58.42 90)
 			(effects
@@
 			)
 		)
-		(property "Description" ""
-			(at 92.71 64.77 0)
-			(effects
-				(font
-					(size 1.27 1.27)
-				)
-				(hide yes)
+		(property "Description" "R_RESET1"
+			(at 92.964 67.056 90)
+			(effects
+				(font
+					(size 1.27 1.27)
+				)
 			)
 		)
@@
 			(project "power_motherboard"
 				(path "/e63e39d7-6ac0-4ffd-8aa3-1841a4541b55/fdc48edb-4989-401e-a47f-b3b658706075"
-					(reference "R_RESET1")
+					(reference "R3")
 					(unit 1)
 				)
@@
 	(symbol
 		(lib_id "Device:C")
-		(at 29.21 60.96 90)
+		(at 44.45 66.04 180)
 		(unit 1)
 		(exclude_from_sim no)
@@
 		(fields_autoplaced yes)
 		(property "Reference" "C1"
-			(at 29.21 53.34 90)
-			(effects
-				(font
-					(size 1.27 1.27)
-				)
+			(at 48.26 64.7699 0)
+			(effects
+				(font
+					(size 1.27 1.27)
+				)
+				(justify right)
 			)
 		)
 		(property "Value" "22pF"
-			(at 29.21 55.88 90)
-			(effects
-				(font
-					(size 1.27 1.27)
-				)
+			(at 48.26 67.3099 0)
+			(effects
+				(font
+					(size 1.27 1.27)
+				)
+				(justify right)
 			)
 		)
 		(property "Footprint" "Capacitor_SMD:C_0603_1608Metric"
-			(at 33.02 59.9948 0)
+			(at 43.4848 62.23 0)
 			(effects
 				(font
@@
 		)
 		(property "Datasheet" "~"
-			(at 29.21 60.96 0)
+			(at 44.45 66.04 0)
 			(effects
 				(font
@@
 		)
 		(property "Description" ""
-			(at 29.21 60.96 0)
+			(at 44.45 66.04 0)
 			(effects
 				(font
@@
 		(on_board yes)
 		(dnp no)
-		(fields_autoplaced yes)
-		(property "Reference" "R_CAN1"
+		(property "Reference" "R2"
 			(at 138.43 46.99 0)
 			(effects
@@
 			)
 		)
-		(property "Description" ""
-			(at 135.89 48.26 0)
-			(effects
-				(font
-					(size 1.27 1.27)
-				)
-				(hide yes)
+		(property "Description" "R_CAN1"
+			(at 142.24 51.562 0)
+			(effects
+				(font
+					(size 1.27 1.27)
+				)
 			)
 		)
@@
 			(project "power_motherboard"
 				(path "/e63e39d7-6ac0-4ffd-8aa3-1841a4541b55/fdc48edb-4989-401e-a47f-b3b658706075"
-					(reference "R_CAN1")
+					(reference "R2")
 					(unit 1)
 				)
