File: raspi_motherboard/power.kicad_sch (KiCad schematic)
At the start: 30 parts, among them J3 Conn_01x03, U3 TPS563200

Commit message: Last update
Parts:
- removed Q_P12VP_1: 2N3906, Package_TO_SOT_SMD:SOT-23, symbol Transistor_BJT:2N3906
- added Q_P12VE_2: 2N3906, Package_TO_SOT_SMD:SOT-23, symbol Transistor_BJT:2N3906
Connections:
- net 12VP_SEC_1: no longer R_12VP_2.1
- net 12VP_SEC_2: now also R_12VP_2.1, Q_P12VE_2.3 (C)
- net at D_12VE_INV1.1 (K), F_12VE1.1, Q_12VP_1.1 (S)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: now also Q_P12VE_1.2 (E); no longer Q_P12VE_1.1 (E)
- net at D_12VE_OT1.1 (K), R_12VE_1.2: now also Q_P12VE_1.1 (B); no longer Q_P12VE_1.2 (B)
- net at D_12VP_INV1.1 (K), F_12VP1.1, Q_12VP_2.1 (S)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: now also Q_P12VE_2.2 (E)
- net at D_12VP_OT1.1 (K), R_12VP_1.2: now also Q_P12VE_2.1 (B)
Changed lines of the file:
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@@
 	)
 	(junction
-		(at 105.41 81.28)
-		(diameter 0)
-		(color 0 0 0 0)
-	)
-	(junction
 		(at 85.09 55.88)
 		(diameter 0)
@@
 	)
 	(junction
+		(at 85.09 83.82)
+		(diameter 0)
+		(color 0 0 0 0)
+	)
+	(junction
 		(at 69.85 43.18)
 		(diameter 0)
@@
 	(wire
 		(pts
-			(xy 85.09 85.09) (xy 105.41 85.09)
-		)
-		(stroke
-			(width 0)
-			(type default)
-		)
-	)
-	(wire
-		(pts
 			(xy 69.85 81.28) (xy 69.85 83.82)
 		)
@@
 	(wire
 		(pts
+			(xy 85.09 83.82) (xy 85.09 85.09)
+		)
+		(stroke
+			(width 0)
+			(type default)
+		)
+	)
+	(wire
+		(pts
 			(xy 109.22 66.04) (xy 109.22 68.58)
 		)
@@
 	(wire
 		(pts
+			(xy 74.93 78.74) (xy 77.47 78.74)
+		)
+		(stroke
+			(width 0)
+			(type default)
+		)
+	)
+	(wire
+		(pts
 			(xy 53.34 57.15) (xy 53.34 64.77)
 		)
@@
 	(wire
 		(pts
-			(xy 77.47 78.74) (xy 77.47 81.28)
+			(xy 74.93 78.74) (xy 74.93 81.28)
 		)
 		(stroke
@@
 	(wire
 		(pts
-			(xy 105.41 85.09) (xy 105.41 81.28)
-		)
-		(stroke
-			(width 0)
-			(type default)
-		)
-	)
-	(wire
-		(pts
 			(xy 69.85 78.74) (xy 69.85 81.28)
 		)
@@
 	(wire
 		(pts
-			(xy 69.85 81.28) (xy 77.47 81.28)
+			(xy 69.85 81.28) (xy 74.93 81.28)
 		)
 		(stroke
@@
 	)
 	(symbol
-		(lib_id "Transistor_BJT:2N3906")
-		(at 82.55 78.74 0)
-		(mirror x)
-		(unit 1)
-		(exclude_from_sim no)
-		(in_bom yes)
-		(on_board yes)
-		(dnp no)
-		(property "Reference" "Q_P12VP_1"
-			(at 91.44 77.47 0)
-			(effects
-				(font
-					(size 1.27 1.27)
-				)
-				(justify left)
-			)
-		)
-		(property "Value" "2N3906"
-			(at 91.44 80.01 0)
-			(effects
-				(font
-					(size 1.27 1.27)
-				)
-				(justify left)
-			)
-		)
-		(property "Footprint" "Package_TO_SOT_SMD:SOT-23"
-			(at 87.63 76.835 0)
-			(effects
-				(font
-					(size 1.27 1.27)
-					(italic yes)
-				)
-				(justify left)
-				(hide yes)
-			)
-		)
-		(property "Datasheet" "https://www.mouser.fr/datasheet/2/308/MMBT3906LT1_D-1811957.pdf"
-			(at 82.55 78.74 0)
-			(effects
-				(font
-					(size 1.27 1.27)
-				)
-				(justify left)
-				(hide yes)
-			)
-		)
-		(property "Description" ""
-			(at 82.55 78.74 0)
-			(effects
-				(font
-					(size 1.27 1.27)
-				)
-				(hide yes)
-			)
-		)
-		(pin "1"
-		)
-		(pin "2"
-		)
-		(pin "3"
-		)
-		(instances
-			(project "power_motherboard"
-				(path "/e63e39d7-6ac0-4ffd-8aa3-1841a4541b55/4c6639a9-406a-464b-9012-e90cb018ad22"
-					(reference "Q_P12VP_1")
-					(unit 1)
-				)
-			)
-		)
-	)
-	(symbol
 		(lib_id "Device:R")
 		(at 69.85 46.99 0)
@@
 	)
 	(symbol
+		(lib_name "2N3906_2")
+		(lib_id "Transistor_BJT:2N3906")
+		(at 82.55 78.74 0)
+		(mirror x)
+		(unit 1)
+		(exclude_from_sim no)
+		(in_bom yes)
+		(on_board yes)
+		(dnp no)
+		(property "Reference" "Q_P12VE_2"
+			(at 87.63 77.47 0)
+			(effects
+				(font
+					(size 1.27 1.27)
+				)
+				(justify left)
+			)
+		)
+		(property "Value" "2N3906"
+			(at 87.63 80.01 0)
+			(effects
+				(font
+					(size 1.27 1.27)
+				)
+				(justify left)
+			)
+		)
+		(property "Footprint" "Package_TO_SOT_SMD:SOT-23"
+			(at 87.63 76.835 0)
+			(effects
+				(font
+					(size 1.27 1.27)
+					(italic yes)
+				)
+				(justify left)
+				(hide yes)
+			)
+		)
+		(property "Datasheet" "https://www.mouser.fr/datasheet/2/308/MMBT3906LT1_D-1811957.pdf"
+			(at 82.55 78.74 0)
+			(effects
+				(font
+					(size 1.27 1.27)
+				)
+				(justify left)
+				(hide yes)
+			)
+		)
+		(property "Description" ""
+			(at 82.55 78.74 0)
+			(effects
+				(font
+					(size 1.27 1.27)
+				)
+				(hide yes)
+			)
+		)
+		(pin "1"
+		)
+		(pin "2"
+		)
+		(pin "3"
+		)
+		(instances
+			(project "power_motherboard"
+				(path "/e63e39d7-6ac0-4ffd-8aa3-1841a4541b55/4c6639a9-406a-464b-9012-e90cb018ad22"
+					(reference "Q_P12VE_2")
+					(unit 1)
+				)
+			)
+		)
+	)
+	(symbol
 		(lib_id "Device:R")
 		(at 92.71 74.93 0)
@@
 	)
 	(symbol
+		(lib_name "2N3906_2")
 		(lib_id "Transistor_BJT:2N3906")
 		(at 82.55 50.8 0)
