File: raspi_motherboard/power_motherboard/power_motherboard.kicad_pcb (KiCad board)
At the start: 4 copper layers, 65 x 59.9 mm, 62 parts, among them J1 GPIO, J2 Conn_02x04_Top_Bottom, J3 Conn_01x03, U1 MCP2515-xST, U2 SN65HVD230, U3 TPS563200, Y1 AMB8-12Mhz

Commit message: Last update
Parts:
- removed Q_P12VE_2: 2N3906, Package_TO_SOT_SMD:SOT-23
- added Q_P12VP_1: 2N3906, Package_TO_SOT_SMD:SOT-23, B.Cu at (127.2, 90.2)
- moved R_12VP_2 9.38 mm to (127.0, 86.9), turned to 0 degrees
- moved D_12VE_OT1 4.40 mm to (109.2, 93.1), turned to 180 degrees
- moved R_12VP_1 3.89 mm to (130.0, 89.8), turned to -90 degrees
- moved D_12VP_OT1 3.56 mm to (130.0, 92.7), turned to -90 degrees
- moved J3 2.25 mm to (122.7, 91.5)
- moved R_12VP_3 2.02 mm to (124.5, 87.8), turned to 90 degrees
- moved R_12VE_1 1.55 mm to (112.5, 93.1), turned to 180 degrees
- moved Q_P12VE_1 0.19 mm to (111.0, 89.8)
Connections:
- Q_P12VE_1 pad 1: Net-(D_12VE_OT1-K) -> Net-(D_12VE_INV1-K)
- Q_P12VE_1 pad 2: Net-(D_12VE_INV1-K) -> Net-(D_12VE_OT1-K)
- R_12VP_2 pad 1: 12VP_SEC_2 -> 12VP_SEC_1
Routing:
- net 12VP_SEC_1: track 2.05 -> 8.80 mm
- net GND_POW: track 24.8 -> 30.3 mm, vias 4 -> 12
- net Net-(D_12VP_INV1-K): track 19.1 -> 23.5 mm, vias 0 -> 1
- net Net-(D_12VP_OT1-K): track 6.10 -> 4.17 mm
- net 12VP_SEC_2: track 5.83 -> 4.11 mm
- net R_IO16: track 22.7 -> 24.1 mm
- net Net-(D_12VE_INV1-K): track 18.4 -> 19.4 mm
- net Net-(D_12VE_OT1-K): track 3.87 -> 4.47 mm
- net GND_ELEC: track 253.2 -> 253.7 mm
